File: Schematics (Eletrical)/PSU/PSU.brd (EAGLE design)
At the start: 99.1 x 79.8 mm, 35 parts, among them IC2 REF02Z, X1 5566-20

Commit message: Update May/2016
Connections:
- net -12V: now also D4.K
Routing:
- net +5.0V: track 200.0 -> 107.6 mm, vias 1 -> 2
- net -12V: track 199.4 -> 280.9 mm, vias 2 -> 4
- added copper zone on layer 1, net +5.0V
- removed copper zone on layer 1, net +5V
Other:
- board text added: "ModSx 2.0 - PSU & ProtoPCB - V0.2 - MachineHum (R.Walker)"
- board text removed: "ModSx 2.0 - PSU & ProtoPCB - V0.1 - MachineHum (R.Walker)"
Changed lines of the file:
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@@
 <?xml version="1.0" encoding="utf-8"?>
 <!DOCTYPE eagle SYSTEM "eagle.dtd">
-<eagle version="6.5.0">
+<eagle version="6.6.0">
 <drawing>
 <settings>
@@
 <hole x="4.064" y="4.064" drill="2.8"/>
 <hole x="94.996" y="4.064" drill="2.8"/>
-<text x="49.53" y="78.5495" size="0.8128" layer="21" font="vector" align="bottom-center">ModSx 2.0 - PSU &amp; ProtoPCB - V0.1 - MachineHum (R.Walker)</text>
+<text x="49.53" y="78.5495" size="0.8128" layer="21" font="vector" align="bottom-center">ModSx 2.0 - PSU &amp; ProtoPCB - V0.2 - MachineHum (R.Walker)</text>
 <text x="70.00875" y="12.54125" size="1.778" layer="25" rot="R90" align="center">B1</text>
 <text x="70.1675" y="19.52625" size="1.778" layer="25" rot="R90" align="center">B2</text>
@@
 <wire x1="12.54125" y1="69.37375" x2="12.54125" y2="71.755" width="0.6096" layer="16"/>
 <wire x1="12.54125" y1="71.755" x2="14.76375" y2="73.9775" width="0.6096" layer="16"/>
-<wire x1="70.6425" y1="44.7675" x2="73.279" y2="44.7675" width="1.016" layer="16"/>
-<wire x1="73.279" y1="44.7675" x2="82.45475" y2="53.94325" width="1.016" layer="16"/>
-<wire x1="82.45475" y1="53.94325" x2="94.5515" y2="66.04" width="1.016" layer="16"/>
-<wire x1="57.531" y1="6.477" x2="59.436" y2="8.382" width="0.254" layer="1"/>
-<wire x1="57.531" y1="5.715" x2="57.531" y2="6.477" width="0.254" layer="1"/>
-<wire x1="58.293" y1="4.953" x2="57.531" y2="5.715" width="0.254" layer="1"/>
-<wire x1="70.485" y1="4.953" x2="58.293" y2="4.953" width="0.254" layer="1"/>
-<wire x1="70.485" y1="44.577" x2="70.485" y2="4.953" width="0.254" layer="1"/>
-<wire x1="59.436" y1="8.382" x2="59.69" y2="8.73125" width="0.254" layer="1"/>
-<wire x1="70.485" y1="44.577" x2="70.6425" y2="44.7675" width="0.254" layer="1"/>
-<wire x1="83.058" y1="53.721" x2="89.154" y2="47.625" width="0.254" layer="16"/>
-<wire x1="82.677" y1="53.721" x2="83.058" y2="53.721" width="0.254" layer="16"/>
-<wire x1="89.154" y1="47.625" x2="89.37625" y2="47.625" width="0.254" layer="16"/>
-<wire x1="82.677" y1="53.721" x2="82.45475" y2="53.94325" width="0.254" layer="16"/>
+<polygon width="0.4064" layer="1" isolate="0.3048">
+<vertex x="1.905" y="1.5875"/>
+<vertex x="1.905" y="4.445"/>
+<vertex x="1.74625" y="77.94625"/>
+<vertex x="97.155" y="77.94625"/>
+<vertex x="97.155" y="1.5875"/>
+</polygon>
+<wire x1="94.5515" y1="66.04" x2="94.5515" y2="62.64275" width="1.016" layer="16"/>
+<wire x1="94.5515" y1="62.64275" x2="92.154375" y2="60.245625" width="1.016" layer="16"/>
+<via x="92.154375" y="60.245625" extent="1-16" drill="0.6" shape="square"/>
+<wire x1="92.154375" y1="60.245625" x2="92.075" y2="60.16625" width="1.016" layer="1"/>
 </signal>
 <signal name="SPARE1">
@@
 <wire x1="59.436" y1="14.097" x2="59.69" y2="13.81125" width="0.254" layer="1"/>
 <wire x1="45.72" y1="44.196" x2="45.56" y2="44.45" width="0.254" layer="1"/>
+<contactref element="D4" pad="K"/>
+<wire x1="91.7575" y1="32.86125" x2="93.6625" y2="32.86125" width="0.4064" layer="1"/>
+<wire x1="93.6625" y1="32.86125" x2="93.6625" y2="8.41375" width="0.4064" layer="1"/>
+<wire x1="93.6625" y1="8.41375" x2="88.185625" y2="8.41375" width="0.4064" layer="1"/>
+<wire x1="88.185625" y1="8.41375" x2="88.185625" y2="7.223125" width="0.4064" layer="1"/>
+<via x="88.185625" y="7.223125" extent="1-16" drill="0.6" shape="square"/>
+<wire x1="88.185625" y1="7.223125" x2="83.02625" y2="7.223125" width="0.4064" layer="16"/>
+<via x="83.02625" y="7.223125" extent="1-16" drill="0.6" shape="square"/>
+<wire x1="83.02625" y1="7.223125" x2="71.27875" y2="7.223125" width="0.4064" layer="1"/>
+<wire x1="71.27875" y1="7.223125" x2="71.27875" y2="3.571875" width="0.4064" layer="1"/>
+<wire x1="71.27875" y1="3.571875" x2="56.67375" y2="3.571875" width="0.4064" layer="1"/>
+<wire x1="56.67375" y1="3.571875" x2="56.67375" y2="13.731875" width="0.4064" layer="1"/>
+<wire x1="56.67375" y1="13.731875" x2="59.69" y2="13.731875" width="0.4064" layer="1"/>
+<wire x1="59.69" y1="13.731875" x2="59.69" y2="13.81125" width="0.4064" layer="1"/>
 </signal>
 <signal name="I2CSCL">
@@
 <wire x1="55.245" y1="67.818" x2="55.5125" y2="67.52" width="0.254" layer="16"/>
 </signal>
-<signal name="+5V">
-<polygon width="0.4064" layer="1" isolate="0.3048">
-<vertex x="1.905" y="1.5875"/>
-<vertex x="1.905" y="4.445"/>
-<vertex x="1.74625" y="77.94625"/>
-<vertex x="97.155" y="77.94625"/>
-<vertex x="97.155" y="1.5875"/>
-</polygon>
-</signal>
 </signals>
